File: hardware/jlink_to_tag/rev_d/jlink_to_tag.sch (EAGLE design)
At the start: 39 parts, among them J2 JLINK_6PIN_TAG-CON, J3 JLINK_6PIN_TAG-CON, J4 JLINK_6PIN_TAG-CON, J5 JLINK_6PIN_TAG-CON, J6 JLINK_6PIN_TAG-CON, J7 JLINK_6PIN_TAG-CON, J8 JLINK_6PIN_TAG-CON, J9 JLINK_6PIN_TAG-CON, U1 LT1763CS8-3.3

Commit message: getting more traces in
Parts:
- added D2, D3, D4, D5, D6, D7, D8, D9: BLUE, SparkFun-LED:LED-BLUE0603
- added R10, R11, R12, R13, R14, R15, R16, R9: 470, SparkFun-Passives:RESISTOR0603-RES
- added S10, S20, S4, S5, S6, S7, S8, S9: PTS645SM43SMTR92, switches:PTS645SM43SMTR92
Connections:
- new net N$10: D8.C, R15.1
- new net N$11: D9.C, R16.1
- new net N$2: D2.C, R9.1
- new net N$5: D3.C, R10.1
- new net N$6: D4.C, R11.1
- new net N$7: D5.C, R12.1
- new net N$8: D6.C, R13.1
- new net N$9: D7.C, R14.1
- net !RST0: now also S4.P$2
- net !RST1: now also S5.P$2
- net !RST2: now also S6.P$2
- net !RST3: now also S7.P$2
- net !RST4: now also S8.P$2
- net !RST5: now also S9.P$2
- net !RST6: now also S10.P$2
- net !RST7: now also S20.P$2
- net EN0: now also D2.A
- net EN1: now also D3.A
- net EN2: now also D4.A
- net EN3: now also D5.A
- net EN4: now also D6.A
- net EN5: now also D7.A
- net EN6: now also D8.A
- net EN7: now also D9.A
- net GND: now also R10.2, R11.2, R12.2, R13.2, R14.2, R15.2, R16.2, R9.2, S10.P$1, S20.P$1, S4.P$1, S5.P$1, S6.P$1, S7.P$1, S8.P$1, S9.P$1

Commit message: board layout
Parts:
- removed C1, C2: 0.01uF, resistor:C-EUC0603
- removed C3: 10uF, SparkFun-Passives:CAP_POL1206
- removed S1: EVQP2, switches:EVQP2
- removed S2, S3: TE_SSA12/SPDT, switches:TE_SSA12/SPDT
- added C4: 10nF, passives:CAPACITOR0603_CAP
- added C5, C6: 4.7uF, passives:CAPACITOR0603_CAP
- added J15: (no value), pinhead:PINHD-2X3
- added S21, S22: STS121PC04, switches:STS121PC04
- added U2: MAX8887EZK33+T, chips:MAX8887EZK33+T
- U1: value LT1763CS8-3.3 -> 74HC4002PW; device linear-technology:LT1763CS8-3.3 -> chips:74HC4002PW; DIGIKEY LT1763CS8-3.3#TRPBFCT-ND -> (none)
Connections:
- removed net N$4: C2.2, U1.BYP
- new net N$1: C4.1, U2.BP
- new net N$15: U1.AOUT, U1.B4
- net !RST: now also J15.3, S22.1; no longer S1.P$1, S3.A
- net 3V3: now also C6.1, S21.1, U1.VCC, U2.OUT; no longer C2.1, C3.+, S2.A, U1.OUT, U1.SENSE
- net 5V: now also C5.1, U2.!SHDN, U2.IN; no longer C1.1, U1.!SHDN, U1.IN
- net EN0: now also U1.BOUT
- net EN1: now also U1.A1
- net EN2: now also U1.A2
- net EN3: now also U1.A3
- net EN4: now also U1.A4
- net EN5: now also U1.B1
- net EN6: now also U1.B2
- net EN7: now also U1.B3
- net GND: now also C4.2, C5.2, C6.2, J15.5, U1.GND, U2.GND; no longer C1.2, C3.-, S1.P$2, U1.GND@1, U1.GND@2, U1.GND@3
- net SWDCLK: now also J15.4
- net SWDIO: now also J15.2, S22.2; no longer S3.IN
- net SWO: now also J15.6
- net VTREF: now also J15.1, S21.2; no longer S2.IN
Other:
- note added: "Reset Buttons"
- note added: "Single-hot Enable Lines"
- note added: "Tag Connect Port Enable Circuits"
- note removed: "3.3 V"
- note removed: "Manual Reset"
- moved on the sheet: S11G$1, S11G$2, S11G$3, S11G$4, S12G$1, S12G$2, S12G$3, S12G$4, S13G$1, S13G$2, S13G$3, S13G$4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

Commit message: started renumber rev d
Parts:
- R10, R11, R12, R13, R14, R15, R16: value 470 -> 1k
- R2, R3, R4, R5, R6, R7, R8: value 1k -> 470
- renumbered C4 to C1, C5 to C2, C6 to C3
Connections:
- net EN1: now also R10.1; no longer R2.1
- net EN2: now also R11.1; no longer R3.1
- net EN3: now also R12.1; no longer R4.1
- net EN4: now also R13.1; no longer R5.1
- net EN5: now also R14.1; no longer R6.1
- net EN6: now also R15.1; no longer R7.1
- net EN7: now also R16.1; no longer R8.1
- net N$10: now also R8.1; no longer R15.1
- net N$11: now also R9.1; no longer R16.1
- net N$2: now also R2.1; no longer R9.1
- net N$5: now also R3.1; no longer R10.1
- net N$6: now also R4.1; no longer R11.1
- net N$7: now also R5.1; no longer R12.1
- net N$8: now also R6.1; no longer R13.1
- net N$9: now also R7.1; no longer R14.1
Other:
- moved on the sheet: R10, R11, R12, R13, R14, R15, R16, R2, R3, R4, R5, R6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

Commit message: Order switches
Parts:
- removed S20: PTS645SM43SMTR92, switches:PTS645SM43SMTR92
- removed S21, S22: STS121PC04, switches:STS121PC04
- added S1, S2, S3: PTS645SM43SMTR92, switches:PTS645SM43SMTR92
- S10: value PTS645SM43SMTR92 -> SN74AHC4066-RGY; device switches:PTS645SM43SMTR92 -> switches:SN74AHC4066-RGY
- S18: value SN74AHC4066-RGY -> STS121PC04; device switches:SN74AHC4066-RGY -> switches:STS121PC04
- S19: value RM100772BCB -> STS121PC04; device switches:RM100772BCB -> switches:STS121PC04
- S9: value PTS645SM43SMTR92 -> RM100772BCB; device switches:PTS645SM43SMTR92 -> switches:RM100772BCB
Connections:
- net !RST: now also S10G$4.IN, S19.1; no longer S18G$4.IN, S22.1
- net !RST0: now also S1.P$2, S10G$4.A; no longer S11G$4.A, S4.P$2
- net !RST1: now also S11G$4.A, S2.P$2; no longer S12G$4.A, S5.P$2
- net !RST2: now also S12G$4.A, S3.P$2; no longer S13G$4.A, S6.P$2
- net !RST3: now also S13G$4.A, S4.P$2; no longer S14G$4.A, S7.P$2
- net !RST4: now also S14G$4.A, S5.P$2; no longer S15G$4.A, S8.P$2
- net !RST5: now also S15G$4.A, S6.P$2; no longer S16G$4.A, S9.P$2
- net !RST6: now also S16G$4.A, S7.P$2; no longer S10.P$2, S17G$4.A
- net !RST7: now also S17G$4.A, S8.P$2; no longer S18G$4.A, S20.P$2
- net 3V3: now also S10G$5.VCC, S18.1, S9.INPUT; no longer S18G$5.VCC, S19.INPUT, S21.1
- net EN0: now also S10G$1.CTRL, S10G$2.CTRL, S10G$3.CTRL, S10G$4.CTRL; no longer S11G$1.CTRL, S11G$2.CTRL, S11G$3.CTRL, S11G$4.CTRL
- net EN1: now also S11G$1.CTRL, S11G$2.CTRL, S11G$3.CTRL, S11G$4.CTRL, S9.A; no longer S12G$1.CTRL, S12G$2.CTRL, S12G$3.CTRL, S12G$4.CTRL, S19.A
- net EN2: now also S12G$1.CTRL, S12G$2.CTRL, S12G$3.CTRL, S12G$4.CTRL, S9.B; no longer S13G$1.CTRL, S13G$2.CTRL, S13G$3.CTRL, S13G$4.CTRL, S19.B
- net EN3: now also S13G$1.CTRL, S13G$2.CTRL, S13G$3.CTRL, S13G$4.CTRL, S9.C; no longer S14G$1.CTRL, S14G$2.CTRL, S14G$3.CTRL, S14G$4.CTRL, S19.C
- net EN4: now also S14G$1.CTRL, S14G$2.CTRL, S14G$3.CTRL, S14G$4.CTRL, S9.D; no longer S15G$1.CTRL, S15G$2.CTRL, S15G$3.CTRL, S15G$4.CTRL, S19.D
- net EN5: now also S15G$1.CTRL, S15G$2.CTRL, S15G$3.CTRL, S15G$4.CTRL, S9.E; no longer S16G$1.CTRL, S16G$2.CTRL, S16G$3.CTRL, S16G$4.CTRL, S19.E
- net EN6: now also S16G$1.CTRL, S16G$2.CTRL, S16G$3.CTRL, S16G$4.CTRL, S9.F; no longer S17G$1.CTRL, S17G$2.CTRL, S17G$3.CTRL, S17G$4.CTRL, S19.F
- net EN7: now also S17G$1.CTRL, S17G$2.CTRL, S17G$3.CTRL, S17G$4.CTRL, S9.G; no longer S18G$1.CTRL, S18G$2.CTRL, S18G$3.CTRL, S18G$4.CTRL, S19.G
- net GND: now also S1.P$1, S10G$5.GND, S2.P$1, S3.P$1; no longer S10.P$1, S18G$5.GND, S20.P$1, S9.P$1
- net SWDCLK: now also S10G$2.IN; no longer S18G$2.IN
- net SWDCLK0: now also S10G$2.A; no longer S11G$2.A
- net SWDCLK1: now also S11G$2.A; no longer S12G$2.A
- net SWDCLK2: now also S12G$2.A; no longer S13G$2.A
- net SWDCLK3: now also S13G$2.A; no longer S14G$2.A
- net SWDCLK4: now also S14G$2.A; no longer S15G$2.A
- net SWDCLK5: now also S15G$2.A; no longer S16G$2.A
- net SWDCLK6: now also S16G$2.A; no longer S17G$2.A
- net SWDCLK7: now also S17G$2.A; no longer S18G$2.A
- net SWDIO: now also S10G$1.IN, S19.2; no longer S18G$1.IN, S22.2
- net SWDIO0: now also S10G$1.A; no longer S11G$1.A
- net SWDIO1: now also S11G$1.A; no longer S12G$1.A
- net SWDIO2: now also S12G$1.A; no longer S13G$1.A
- net SWDIO3: now also S13G$1.A; no longer S14G$1.A
- net SWDIO4: now also S14G$1.A; no longer S15G$1.A
- net SWDIO5: now also S15G$1.A; no longer S16G$1.A
- net SWDIO6: now also S16G$1.A; no longer S17G$1.A
- net SWDIO7: now also S17G$1.A; no longer S18G$1.A
- net SWO: now also S10G$3.IN; no longer S18G$3.IN
- net SWO0: now also S10G$3.A; no longer S11G$3.A
- net SWO1: now also S11G$3.A; no longer S12G$3.A
- net SWO2: now also S12G$3.A; no longer S13G$3.A
- net SWO3: now also S13G$3.A; no longer S14G$3.A
- net SWO4: now also S14G$3.A; no longer S15G$3.A
- net SWO5: now also S15G$3.A; no longer S16G$3.A
- net SWO6: now also S16G$3.A; no longer S17G$3.A
- net SWO7: now also S17G$3.A; no longer S18G$3.A
- net VTREF: now also S18.2; no longer S21.2
Other:
- moved on the sheet: S11G$1, S11G$2, S11G$3, S11G$4, S12G$1, S12G$2, S12G$3, S12G$4, S13G$1, S13G$2, S13G$3, S13G$4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
